File: ypvs.kicad_pcb (KiCad board)
At the start: 2 copper layers, 60 x 55 mm, 23 parts, among them J1 Servo, J2 LM_2596 _Input, J3 HV_Cable, J4 Motorcycle Battery, J5 Debug UART, U1 Stm32f103_BluePill, U2 LM1117-3.3, U3 H11L1

Commit message: Final v01
Parts:
- moved J4 2.54 mm to (18.8, 114.8), turned to 180 degrees
- moved U2 0.53 mm to (47.4, 114.8)
- moved J5 0.51 mm to (33.0, 115.8)
Routing:
- net +12V: track 38.9 -> 42.3 mm
- net +3V3: track 81.1 -> 80.4 mm
Changed lines of the file:
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@@
     (thickness 1.6)
     (drawings 17)
-    (tracks 78)
+    (tracks 77)
     (zones 0)
     (modules 23)
@@
   (layers
     (0 F.Cu signal hide)
-    (31 B.Cu signal hide)
+    (31 B.Cu signal)
     (32 B.Adhes user)
     (33 F.Adhes user)
@@
   )
   (setup
-    (last_trace_width 1.524)
+    (last_trace_width 0.508)
     (user_trace_width 0.254)
     (user_trace_width 0.381)
@@
     (visible_elements 7FFFFFFF)
     (pcbplotparams
-      (layerselection 0x010fc_ffffffff)
+      (layerselection 0x010f0_ffffffff)
       (usegerberextensions false)
       (usegerberattributes true)
@@
       (psa4output false)
       (plotreference true)
-      (plotvalue true)
+      (plotvalue false)
       (plotinvisibletext false)
       (padsonsilk false)
@@
       (outputformat 1)
       (mirror false)
-      (drillshape 1)
+      (drillshape 0)
       (scaleselection 1)
-      (outputdirectory ""))
+      (outputdirectory "gerbers/"))
   )
   (net 0 "")
@@
   )
   (module Connector_PinHeader_2.54mm:PinHeader_1x02_P2.54mm_Vertical (layer F.Cu)
-    (at 18.796 112.268)
+    (at 18.796 114.808 180)
     (descr "Through hole straight pin header, 1x02, 2.54mm pitch, single row")
     (tags "Through hole pin header THT 1x02 2.54mm single row")
@@
       (effects (font (size 1 1) (thickness 0.15)))
     )
-    (pad 1 thru_hole rect (at 0 0) (size 1.7 1.7) (drill 1) (layers *.Cu *.Mask)
+    (pad 1 thru_hole rect (at 0 0 180) (size 1.7 1.7) (drill 1) (layers *.Cu *.Mask)
       (net 1 GND))
-    (pad 2 thru_hole oval (at 0 2.54) (size 1.7 1.7) (drill 1) (layers *.Cu *.Mask)
+    (pad 2 thru_hole oval (at 0 2.54 180) (size 1.7 1.7) (drill 1) (layers *.Cu *.Mask)
       (net 2 +12V))
     (model ${KISYS3DMOD}/Connector_PinHeader_2.54mm.3dshapes/PinHeader_1x02_P2.54mm_Vertical.wrl
@@
   )
   (module Package_TO_SOT_SMD:SOT-223-3_TabPin2 (layer B.Cu)
-    (at 47.244 115.316 90)
+    (at 47.4 114.808 90)
     (descr "module CMS SOT223 4 pins")
     (tags "CMS SOT")
@@
   )
   (module Connector_PinHeader_2.54mm:PinHeader_1x02_P2.54mm_Vertical (layer F.Cu)
-    (at 32.512 115.824 270)
+    (at 33.02 115.824 270)
     (descr "Through hole straight pin header, 1x02, 2.54mm pitch, single row")
     (tags "Through hole pin header THT 1x02 2.54mm single row")
@@
     )
   )
-  (gr_text GND (at 18.8 117.6) (layer F.SilkS)
+  (gr_text GND (at 18.796 117.348) (layer F.SilkS)
     (effects (font (size 0.762 0.762) (thickness 0.15)))
   )
-  (gr_text +12V (at 18.6 109.4) (layer F.SilkS)
+  (gr_text +12V (at 18.796 109.728) (layer F.SilkS)
     (effects (font (size 0.762 0.762) (thickness 0.15)))
   )
@@
     (effects (font (size 0.762 0.762) (thickness 0.15)))
   )
-  (gr_text RX (at 32.6 113.2) (layer F.SilkS)
+  (gr_text RX (at 33.108 113.2) (layer F.SilkS)
     (effects (font (size 1 1) (thickness 0.15)))
   )
-  (gr_text TX (at 29.8 113.2) (layer F.SilkS)
+  (gr_text TX (at 30.308 113.2) (layer F.SilkS)
     (effects (font (size 1 1) (thickness 0.15)))
   )
@@
   (segment (start 28.448 74.168) (end 27.94 73.66) (width 1.524) (layer F.Cu) (net 1))
   (segment (start 28.448 76) (end 28.448 74.168) (width 1.524) (layer B.Cu) (net 1))
-  (segment (start 18.796 114.808) (end 22.86 114.808) (width 0.508) (layer B.Cu) (net 2))
-  (segment (start 22.86 114.808) (end 26.416 118.364) (width 0.508) (layer B.Cu) (net 2))
-  (segment (start 26.416 118.364) (end 26.416 121.92) (width 0.508) (layer B.Cu) (net 2))
-  (segment (start 27.432 122.936) (end 28.956 122.936) (width 0.508) (layer B.Cu) (net 2))
-  (segment (start 26.416 121.92) (end 27.432 122.936) (width 0.508) (layer B.Cu) (net 2))
-  (segment (start 28.956 122.936) (end 34.036 122.936) (width 0.508) (layer B.Cu) (net 2))
-  (segment (start 44.944 124.22) (end 44.944 118.466) (width 0.508) (layer B.Cu) (net 2))
-  (segment (start 43.688 125.476) (end 44.944 124.22) (width 0.508) (layer B.Cu) (net 2))
-  (segment (start 34.036 122.936) (end 36.576 125.476) (width 0.508) (layer B.Cu) (net 2))
-  (segment (start 36.576 125.476) (end 43.688 125.476) (width 0.508) (layer B.Cu) (net 2))
-  (segment (start 47.244 112.166) (end 47.244 84.836) (width 0.508) (layer B.Cu) (net 3))
-  (segment (start 52.0954 79.9846) (end 54.5846 79.9846) (width 0.508) (layer B.Cu) (net 3))
-  (segment (start 47.244 84.836) (end 52.0954 79.9846) (width 0.508) (layer B.Cu) (net 3))
-  (segment (start 60.452 123.952) (end 60.452 120.904) (width 0.508) (layer B.Cu) (net 3))
-  (segment (start 49.784 125.476) (end 58.928 125.476) (width 0.508) (layer B.Cu) (net 3))
-  (segment (start 58.928 125.476) (end 60.452 123.952) (width 0.508) (layer B.Cu) (net 3))
-  (segment (start 47.244 118.466) (end 47.244 122.936) (width 0.508) (layer B.Cu) (net 3))
-  (segment (start 47.244 122.936) (end 49.784 125.476) (width 0.508) (layer B.Cu) (net 3))
   (segment (start 60.452 120.904) (end 62.992 118.364) (width 0.508) (layer B.Cu) (net 3))
   (segment (start 62.992 118.364) (end 66.04 118.364) (width 0.508) (layer B.Cu) (net 3))
@@
   (segment (start 37.3634 87.6046) (end 39.3446 87.6046) (width 0.254) (layer F.Cu) (net 46))
   (segment (start 35.052 89.916) (end 37.3634 87.6046) (width 0.254) (layer F.Cu) (net 46))
+  (segment (start 43.688 125.476) (end 44.944 124.22) (width 0.508) (layer B.Cu) (net 2))
+  (segment (start 34.036 122.936) (end 36.576 125.476) (width 0.508) (layer B.Cu) (net 2))
+  (segment (start 36.576 125.476) (end 43.688 125.476) (width 0.508) (layer B.Cu) (net 2))
+  (segment (start 27.432 122.936) (end 34.036 122.936) (width 0.508) (layer B.Cu) (net 2))
+  (segment (start 26.416 115.316) (end 26.416 121.92) (width 0.508) (layer B.Cu) (net 2))
+  (segment (start 18.796 112.268) (end 23.368 112.268) (width 0.508) (layer B.Cu) (net 2))
+  (segment (start 26.416 121.92) (end 27.432 122.936) (width 0.508) (layer B.Cu) (net 2))
+  (segment (start 23.368 112.268) (end 26.416 115.316) (width 0.508) (layer B.Cu) (net 2))
+  (segment (start 44.944 118.114) (end 45.1 117.958) (width 0.508) (layer B.Cu) (net 2))
+  (segment (start 44.944 124.22) (end 44.944 118.114) (width 0.508) (layer B.Cu) (net 2))
+  (segment (start 48.26 125.476) (end 47.4 124.616) (width 0.508) (layer B.Cu) (net 3))
+  (segment (start 58.928 125.476) (end 48.26 125.476) (width 0.508) (layer B.Cu) (net 3))
+  (segment (start 47.4 124.616) (end 47.4 117.958) (width 0.508) (layer B.Cu) (net 3))
+  (segment (start 60.452 120.904) (end 60.452 123.952) (width 0.508) (layer B.Cu) (net 3))
+  (segment (start 60.452 123.952) (end 58.928 125.476) (width 0.508) (layer B.Cu) (net 3))
+  (segment (start 47.4 87.1692) (end 47.4 111.658) (width 0.508) (layer B.Cu) (net 3))
+  (segment (start 54.5846 79.9846) (end 47.4 87.1692) (width 0.508) (layer B.Cu) (net 3))
   (zone (net 1) (net_name GND) (layer F.Cu) (hatch edge 0.508)
     (connect_pads (clearance 0.508))
